Commit message: Fix for mesh filenames

File: rb_theron_description/urdf/bases/theron_base.urdf.xacro (robot description, xacro)
@@ -38,5 +38,5 @@
         <xacro:if value="${hq}">
           <geometry>
-            <mesh filename="package://rb_theron_description/meshes/bases/theron_base.stl"/>
+            <mesh filename="$(find rb_theron_description)/meshes/bases/theron_base.stl"/>
           </geometry>
         </xacro:if>
@@ -55,5 +55,5 @@
         <geometry>
           <!--box size="0.390 0.240 0.165"/-->
-          <mesh filename="package://rb_theron_description/meshes/bases/theron_base.stl"/>
+          <mesh filename="$(find rb_theron_description)/meshes/bases/theron_base.stl"/>
         </geometry>
       </collision>
@@ -69,5 +69,5 @@
         <xacro:if value="${hq}">
           <geometry>
-            <mesh filename="package://rb_theron_description/meshes/bases/mcq_prototype_bottom_cover.dae"/>
+            <mesh filename="$(find rb_theron_description)/meshes/bases/mcq_prototype_bottom_cover.dae"/>
           </geometry>
         </xacro:if>
@@ -84,5 +84,5 @@
         <origin xyz="0 0 0" rpy="0 0 0 " />
         <geometry>
-          <mesh filename="package://rb_theron_description/meshes/bases/mcq_prototype_bottom_cover.dae"/>
+          <mesh filename="$(find rb_theron_description)/meshes/bases/mcq_prototype_bottom_cover.dae"/>
         </geometry>
       </collision>

File: rb_theron_description/urdf/pole/mcq_pole.urdf.xacro (robot description, xacro)
@@ -25,5 +25,5 @@
           <geometry>
             <!-- <box size="0.25 0.25 1.55"/> -->
-            <mesh filename="package://rb_theron_description/meshes/pole/mcq_pole.stl"/>
+            <mesh filename="$(find rb_theron_description)/meshes/pole/mcq_pole.stl"/>
           </geometry>
         <material name="darkgrey">
@@ -35,5 +35,5 @@
         <geometry>
           <!-- <box size="0.25 0.25 1.55"/> -->
-          <mesh filename="package://rb_theron_description/meshes/pole/mcq_pole.stl"/>
+          <mesh filename="$(find rb_theron_description)/meshes/pole/mcq_pole.stl"/>
         </geometry>
       </collision>

File: rb_theron_description/urdf/pole/simple_pole.urdf.xacro (robot description, xacro)
@@ -25,5 +25,5 @@
           <geometry>
             <!-- <box size="0.25 0.25 1.55"/> -->
-            <mesh filename="package://rb_theron_description/meshes/pole/simple_pole.dae"/>
+            <mesh filename="$(find rb_theron_description)/meshes/pole/simple_pole.dae"/>
           </geometry>
         <material name="darkgrey">
@@ -35,5 +35,5 @@
         <geometry>
           <!-- <box size="0.25 0.25 1.55"/> -->
-          <mesh filename="package://rb_theron_description/meshes/pole/simple_pole.dae"/>
+          <mesh filename="$(find rb_theron_description)/meshes/pole/simple_pole.dae"/>
         </geometry>
       </collision>

File: rb_theron_description/urdf/rocker/mcq_prototype_rocker.urdf.xacro (robot description, xacro)
@@ -36,10 +36,10 @@
           <xacro:if value="${reflect}">
             <geometry>
-	          <mesh filename="package://rb_theron_description/meshes/rocker/mcq_prototype_rocker_r.dae" />
+	          <mesh filename="$(find rb_theron_description)/meshes/rocker/mcq_prototype_rocker_r.dae" />
             </geometry>
           </xacro:if>
           <xacro:unless value="${reflect}">
             <geometry>
-              <mesh filename="package://rb_theron_description/meshes/rocker/mcq_prototype_rocker_l.dae" />
+              <mesh filename="$(find rb_theron_description)/meshes/rocker/mcq_prototype_rocker_l.dae" />
             </geometry>
 		  </xacro:unless>
@@ -49,10 +49,10 @@
           <xacro:if value="${reflect}">
             <geometry>
-	          <mesh filename="package://rb_theron_description/meshes/rocker/mcq_prototype_rocker_r.dae" />
+	          <mesh filename="$(find rb_theron_description)/meshes/rocker/mcq_prototype_rocker_r.dae" />
             </geometry>
           </xacro:if>
           <xacro:unless value="${reflect}">
             <geometry>
-              <mesh filename="package://rb_theron_description/meshes/rocker/mcq_prototype_rocker_l.dae" />
+              <mesh filename="$(find rb_theron_description)/meshes/rocker/mcq_prototype_rocker_l.dae" />
             </geometry>
 		  </xacro:unless>

File: rb_theron_description/urdf/wheels/castor.urdf.xacro (robot description, xacro)
@@ -33,5 +33,5 @@
         <origin xyz="0 0 0" rpy="0 0 0" />
           <geometry>
-	       <mesh filename="package://rb_theron_description/meshes/wheels/mcq_prototype_base_castor.dae" />
+	       <mesh filename="$(find rb_theron_description)/meshes/wheels/mcq_prototype_base_castor.dae" />
           </geometry>
       </visual>
@@ -39,5 +39,5 @@
         <origin xyz="0 0 0" rpy="0 0 0" />
           <geometry>
-	       <mesh filename="package://rb_theron_description/meshes/wheels/mcq_prototype_base_castor.dae" />
+	       <mesh filename="$(find rb_theron_description)/meshes/wheels/mcq_prototype_base_castor.dae" />
           </geometry>
       </collision>
@@ -69,5 +69,5 @@
           <origin xyz="0 0 0" rpy="0 0 0" />
           <geometry>
-		<mesh filename="package://rb_theron_description/meshes/wheels/mcq_prototype_castor_wheel.dae" />
+		<mesh filename="$(find rb_theron_description)/meshes/wheels/mcq_prototype_castor_wheel.dae" />
           </geometry>
         </xacro:if -->
@@ -85,5 +85,5 @@
 	  <!-- origin xyz="0 0 0" rpy="0 0 0" / -->
         <geometry>
-		  <!-- mesh filename="package://rb_theron_description/meshes/wheels/mcq_prototype_castor_wheel.dae" / -->
+		  <!-- mesh filename="$(find rb_theron_description)/meshes/wheels/mcq_prototype_castor_wheel.dae" / -->
           <cylinder length="${caster_height}" radius="${caster_radius}" />
           <!-- sphere radius="${caster_radius}"/ -->
