Commit message: Added some ros2_control stuff, which is not fully working now because the connection to gazebo does not work properly.

File: rb_theron_description/urdf/rocker/mcq_prototype_rocker.urdf.xacro (robot description, xacro)
@@ -75,4 +75,25 @@
 	  </actuator>
 	</transmission>
+  <ros2_control name="${prefix}rsupport_joint_ros2_control" type="system">
+			<!-- <hardware>
+				<xacro:if value="${use_fake_hardware}">
+				<plugin>fake_components/GenericSystem</plugin>
+				<param name="fake_sensor_commands">${fake_sensor_commands}</param>
+				<param name="state_following_offset">0.0</param>
+				</xacro:if>
+				<xacro:unless value="${use_fake_hardware}">
+				<plugin>ros2_control_demo_hardware/DiffBotSystemHardware</plugin>
+				<param name="example_param_hw_start_duration_sec">2.0</param>
+				<param name="example_param_hw_stop_duration_sec">3.0</param>
+				</xacro:unless>
+			</hardware> -->
+			<hardware>
+				<plugin>fake_components/GenericSystem</plugin>
+			</hardware>
+			<joint name="${prefix}joint_rsupport">
+				<state_interface name="position"/>
+				<state_interface name="velocity"/>
+			</joint>
+		</ros2_control>
 	<!-- Flag to select the high or low quality model -->
 	<xacro:property name="hq" value="true" />

File: rb_theron_description/urdf/wheels/castor.urdf.xacro (robot description, xacro)
@@ -120,4 +120,46 @@
       </actuator>
     </transmission>
+    <ros2_control name="${prefix}support_joint_ros2_control" type="system">
+			<!-- <hardware>
+				<xacro:if value="${use_fake_hardware}">
+				<plugin>fake_components/GenericSystem</plugin>
+				<param name="fake_sensor_commands">${fake_sensor_commands}</param>
+				<param name="state_following_offset">0.0</param>
+				</xacro:if>
+				<xacro:unless value="${use_fake_hardware}">
+				<plugin>ros2_control_demo_hardware/DiffBotSystemHardware</plugin>
+				<param name="example_param_hw_start_duration_sec">2.0</param>
+				<param name="example_param_hw_stop_duration_sec">3.0</param>
+				</xacro:unless>
+			</hardware> -->
+			<hardware>
+				<plugin>fake_components/GenericSystem</plugin>
+			</hardware>
+			<joint name="${prefix}joint_support">
+				<state_interface name="position"/>
+				<state_interface name="velocity"/>
+			</joint>
+		</ros2_control>
+    <ros2_control name="${prefix}wheel_joint_ros2_control" type="system">
+			<!-- <hardware>
+				<xacro:if value="${use_fake_hardware}">
+				<plugin>fake_components/GenericSystem</plugin>
+				<param name="fake_sensor_commands">${fake_sensor_commands}</param>
+				<param name="state_following_offset">0.0</param>
+				</xacro:if>
+				<xacro:unless value="${use_fake_hardware}">
+				<plugin>ros2_control_demo_hardware/DiffBotSystemHardware</plugin>
+				<param name="example_param_hw_start_duration_sec">2.0</param>
+				<param name="example_param_hw_stop_duration_sec">3.0</param>
+				</xacro:unless>
+			</hardware> -->
+			<hardware>
+				<plugin>fake_components/GenericSystem</plugin>
+			</hardware>
+			<joint name="${prefix}joint_wheel">
+				<state_interface name="position"/>
+				<state_interface name="velocity"/>
+			</joint>
+		</ros2_control>
     <!-- gazebo reference="${prefix}support">
 			<mu1 value="5.0"/>

File: rb_theron_description/urdf/wheels/rubber_wheel.transmission.xacro (robot description, xacro)
@@ -17,4 +17,29 @@
 			</actuator>
 		</transmission>
+		<ros2_control name="${prefix}_wheel_joint_ros2_control" type="system">
+			<!-- <hardware>
+				<xacro:if value="${use_fake_hardware}">
+				<plugin>fake_components/GenericSystem</plugin>
+				<param name="fake_sensor_commands">${fake_sensor_commands}</param>
+				<param name="state_following_offset">0.0</param>
+				</xacro:if>
+				<xacro:unless value="${use_fake_hardware}">
+				<plugin>ros2_control_demo_hardware/DiffBotSystemHardware</plugin>
+				<param name="example_param_hw_start_duration_sec">2.0</param>
+				<param name="example_param_hw_stop_duration_sec">3.0</param>
+				</xacro:unless>
+			</hardware> -->
+			<hardware>
+				<plugin>fake_components/GenericSystem</plugin>
+			</hardware>
+			<joint name="${prefix}_wheel_joint">
+				<command_interface name="velocity">
+				<param name="min">-1</param>
+				<param name="max">1</param>
+				</command_interface>
+				<state_interface name="position"/>
+				<state_interface name="velocity"/>
+			</joint>
+		</ros2_control>
 	</xacro:macro>
 </robot>
