Commit message: rb_theron adjusted to Robast configuration

File: rb_theron_description/robots/rb_theron.urdf.xacro (robot description, xacro)
@@ -64,13 +64,19 @@
 		<origin xyz="0.3305 0.0 0.1468" rpy="0 0 0"/>
 	</xacro:sensor_r430>
+	<xacro:sensor_r430 prefix="$(arg prefix)back_realsense_camera" parent="$(arg prefix)base_link" prefix_topic="back_realsense_camera">
+		<origin xyz="-0.3305 0.0 0.1468" rpy="0 0 3.1416"/>
+	</xacro:sensor_r430>
   <!-- TODO: Moved 0.01 in x, otherwise the camera is still inside the robot -->
-	<xacro:sensor_orbbec_astra prefix="$(arg prefix)front_rgbd_camera" parent="$(arg prefix)base_link" prefix_topic="front_rgbd_camera">
+	<!--xacro:sensor_orbbec_astra prefix="$(arg prefix)front_rgbd_camera" parent="$(arg prefix)base_link" prefix_topic="front_rgbd_camera">
 		<origin xyz="0.3305 0.0 0.1898" rpy="0 0 0"/>
-	</xacro:sensor_orbbec_astra>
+	</xacro:sensor_orbbec_astra -->
 	<xacro:sensor_imu_hector prefix="$(arg prefix)imu" parent="$(arg prefix)base_link">
 		<origin xyz="-0.1975 0.0 0.1598" rpy="0 0 0"/>
 	</xacro:sensor_imu_hector>
-	<xacro:sensor_sick_nanoscan3 prefix="$(arg prefix)front_laser" parent="$(arg prefix)base_link" prefix_topic="front_laser" min_angle="-2.0507619" max_angle="2.0507619">
+	<xacro:sensor_hokuyo_ust20lx prefix="$(arg prefix)front_laser" parent="$(arg prefix)base_link" prefix_topic="front_laser" min_angle="-2.0507619" max_angle="2.0507619">
 		<origin xyz="0.250 0.0 0.1643" rpy="0 3.1416 3.1416"/>
+	</xacro:sensor_hokuyo_ust20lx>
+	<xacro:sensor_sick_nanoscan3 prefix="$(arg prefix)back_laser" parent="$(arg prefix)base_link" prefix_topic="back_laser" min_angle="-2.0507619" max_angle="2.0507619">
+		<origin xyz="-0.250 0.0 0.1643" rpy="0 3.1416 0"/>
 	</xacro:sensor_sick_nanoscan3>
 </robot>

File: rb_theron_description/urdf/bases/theron_base.urdf.xacro (robot description, xacro)
@@ -59,5 +59,5 @@
       </collision>
     </link>
-    <!-- <link name="${prefix}bottom_cover_link">
+   <link name="${prefix}bottom_cover_link">
       <inertial>
         <mass value="2.0" />
@@ -87,10 +87,10 @@
         </geometry>
       </collision>
-    </link> -->
-    <!-- <joint name="${prefix}bottom_cover_joint" type="fixed">
+    </link>
+     <joint name="${prefix}bottom_cover_joint" type="fixed">
        <origin rpy="0 0 0" xyz="0 0 0"/>
        <parent link="${prefix}base_link"/>
        <child link="${prefix}bottom_cover_link"/>
-    </joint> -->
+    </joint>
     <!-- DOCKING CONTACTS -->
     <!--joint name="${prefix}base_docking_joint" type="fixed">

Commit message: Added rs_lidar_16, that is commented out for the moment until we can convert pointcloud to laserscan

File: rb_theron_description/robots/rb_theron.urdf.xacro (robot description, xacro)
@@ -77,4 +77,8 @@
 		<origin xyz="0.250 0.0 0.1643" rpy="0 3.1416 3.1416"/>
 	</xacro:sensor_hokuyo_ust20lx>
+	<!-- Uncomment this as soon as we can convert pointcloud to laserscan -->
+	<!-- <xacro:sensor_rs_lidar_16 prefix="$(arg prefix)front_laser" parent="$(arg prefix)base_link" prefix_topic="front_laser" min_angle="-1.9507619" max_angle="1.9507619">
+		<origin xyz="0.250 0.0 0.1643" rpy="1.57079632679 0 0"/>
+	</xacro:sensor_rs_lidar_16> -->
 	<xacro:sensor_sick_nanoscan3 prefix="$(arg prefix)back_laser" parent="$(arg prefix)base_link" prefix_topic="back_laser" min_angle="-1.8107619" max_angle="1.8107619">
 		<origin xyz="-0.250 0.0 0.1643" rpy="0 3.1416 0"/>

Commit message: Adding module cage to rb theron

File: rb_theron_description/robots/rb_theron.urdf.xacro (robot description, xacro)
@@ -84,3 +84,8 @@
 		<origin xyz="-0.250 0.0 0.1643" rpy="0 3.1416 0"/>
 	</xacro:sensor_sick_nanoscan3> -->
+	<!-- ROBAST Module Cage -->
+	<xacro:include filename="$(find rb_theron_description)/urdf/module_cage/module_cage.urdf.xacro" />
+	<xacro:module_cage prefix="$(arg prefix)module_cage" parent="$(arg prefix)base_link">
+		<origin xyz="-0.18 -0.20 0.2225" rpy="0 0 1.570796326794896619"/>
+	</xacro:module_cage>
 </robot>

Commit message: Added rs_lidar_16 to the theron. Minor placement fix for module cage

File: rb_theron_description/robots/rb_theron.urdf.xacro (robot description, xacro)
@@ -77,8 +77,7 @@
 		<origin xyz="0.250 0.0 0.1643" rpy="0 3.1416 3.1416"/>
 	</xacro:sensor_sick_nanoscan3>
-	<!-- Uncomment this as soon as we can convert pointcloud to laserscan -->
-	<!-- <xacro:sensor_rs_lidar_16 prefix="$(arg prefix)front_laser" parent="$(arg prefix)base_link" prefix_topic="front_laser" min_angle="-1.9507619" max_angle="1.9507619">
-		<origin xyz="0.250 0.0 0.1643" rpy="1.57079632679 0 0"/>
-	</xacro:sensor_rs_lidar_16> -->
+	<xacro:sensor_rs_lidar_16 prefix="$(arg prefix)top_laser" parent="$(arg prefix)base_link" prefix_topic="top_laser" min_angle="-1.9507619" max_angle="1.9507619">
+		<origin xyz="0.214 0.0 0.275" rpy="-1.57079632679 0 -0.23"/>
+	</xacro:sensor_rs_lidar_16>
 	<!-- <xacro:sensor_sick_nanoscan3 prefix="$(arg prefix)back_laser" parent="$(arg prefix)base_link" prefix_topic="back_laser" min_angle="-1.8107619" max_angle="1.8107619">
 		<origin xyz="-0.250 0.0 0.1643" rpy="0 3.1416 0"/>
@@ -87,5 +86,5 @@
 	<xacro:include filename="$(find rb_theron_description)/urdf/module_cage/module_cage.urdf.xacro" />
 	<xacro:module_cage prefix="$(arg prefix)module_cage" parent="$(arg prefix)base_link">
-		<origin xyz="-0.18 -0.20 0.2225" rpy="0 0 1.570796326794896619"/>
+		<origin xyz="-0.18 -0.1997 0.2225" rpy="0 0 1.570796326794896619"/>
 	</xacro:module_cage>
 </robot>

Commit message: xacro und prefix anpassungen

File: rb_theron_description/robots/rb_theron.urdf.xacro (robot description, xacro)
@@ -43,5 +43,5 @@
 	<xacro:theron_base prefix="$(arg prefix)" publish_bf="true" hq="${hq}" />
 	<!-- Gazebo ros control pluggins -->
-	<xacro:ros_control/>
+	<xacro:ros_control prefix="$(arg prefix)"/>
 	<xacro:gazebo_colors prefix="$(arg prefix)"/>
 	<!-- WHEELS -->

File: rb_theron_description/urdf/bases/theron_base.urdf.xacro (robot description, xacro)
@@ -2,9 +2,9 @@
 <robot name="rbogie_base"
   xmlns:xacro="http://www.ros.org/wiki/xacro">
-<macro name="box_inertia_robot" params="m x y z">
+<xacro:macro name="box_inertia_robot" params="m x y z">
         <inertia  ixx="${m*(y*y+z*z)/12}" ixy = "0" ixz = "0"
                   iyy="${m*(x*x+z*z)/12}" iyz = "0"
                   izz="${m*(x*x+z*z)/12}" />
-</macro>
+</xacro:macro>
   <xacro:macro name="theron_base" params="prefix publish_bf hq">
     <!-- Robot mechanical and motor parameters -->

File: rb_theron_description/urdf/common.gazebo.xacro (robot description, xacro)
@@ -2,5 +2,5 @@
 <robot xmlns:xacro="http://www.ros.org/wiki/xacro">
 	<!-- ROS CONTROL GAZEBO PLUGIN -->
-	<xacro:macro name="ros_control">
+	<xacro:macro name="ros_control" params="prefix">
 		<gazebo>
 			<!-- <plugin filename="libgazebo_ros2_control.so" name="gazebo_ros2_control">
@@ -13,16 +13,16 @@
 				<alwaysOn>1</alwaysOn>
 				<update_rate>30</update_rate>
-				<joint_name>leftjoint_rsupport</joint_name>
-				<joint_name>rightjoint_rsupport</joint_name>
-				<joint_name>left_wheel_joint</joint_name>
-				<joint_name>right_wheel_joint</joint_name>
-				<joint_name>leftcastorjoint_support</joint_name>
-				<joint_name>rightcastorjoint_support</joint_name>
-				<joint_name>leftcastorjoint_wheel</joint_name>
-				<joint_name>rightcastorjoint_wheel</joint_name>
-				<joint_name>leftjoint_support</joint_name>
-				<joint_name>rightjoint_support</joint_name>
-				<joint_name>leftjoint_wheel</joint_name>
-				<joint_name>rightjoint_wheel</joint_name>
+				<joint_name>$(arg prefix)leftjoint_rsupport</joint_name>
+				<joint_name>$(arg prefix)rightjoint_rsupport</joint_name>
+				<joint_name>$(arg prefix)left_wheel_joint</joint_name>
+				<joint_name>$(arg prefix)right_wheel_joint</joint_name>
+				<joint_name>$(arg prefix)leftcastorjoint_support</joint_name>
+				<joint_name>$(arg prefix)rightcastorjoint_support</joint_name>
+				<joint_name>$(arg prefix)leftcastorjoint_wheel</joint_name>
+				<joint_name>$(arg prefix)rightcastorjoint_wheel</joint_name>
+				<joint_name>$(arg prefix)leftjoint_support</joint_name>
+				<joint_name>$(arg prefix)rightjoint_support</joint_name>
+				<joint_name>$(arg prefix)leftjoint_wheel</joint_name>
+				<joint_name>$(arg prefix)rightjoint_wheel</joint_name>
 			</plugin>
 			<plugin name="diff_drive" filename="libgazebo_ros_diff_drive.so">
@@ -30,6 +30,6 @@
 				<update_rate>30</update_rate>
 				<!-- wheels -->
-				<left_joint>left_wheel_joint</left_joint>
-				<right_joint>right_wheel_joint</right_joint>
+				<left_joint>$(arg prefix)left_wheel_joint</left_joint>
+				<right_joint>$(arg prefix)right_wheel_joint</right_joint>
 				<!-- kinematics -->
 				<wheel_separation>0.5032</wheel_separation>
@@ -44,6 +44,7 @@
 				<publish_wheel_tf>false</publish_wheel_tf>
 				<odometry_topic>odom</odometry_topic>
-				<odometry_frame>odom</odometry_frame>
-				<base_frame>base_footprint</base_frame>
+				<odometry_frame>$(arg prefix)odom</odometry_frame>
+				<!-- <base_frame>$(arg prefix)base_footprint</base_frame> -->
+    				<robot_base_frame>$(arg prefix)base_footprint</robot_base_frame>
 			</plugin>
 		</gazebo>

File: rb_theron_description/urdf/module_cage/module_cage.urdf.xacro (robot description, xacro)
@@ -1,9 +1,9 @@
 <?xml version="1.0"?>
 <robot name="module_cage" xmlns:xacro="http://www.ros.org/wiki/xacro">
-<macro name="box_inertia_robot" params="m x y z">
+<xacro:macro name="box_inertia_robot" params="m x y z">
 	<inertia  ixx="${m*(y*y+z*z)/12}" ixy = "0" ixz = "0"
 			iyy="${m*(x*x+z*z)/12}" iyz = "0"
 			izz="${m*(x*x+z*z)/12}" />
-</macro>
+</xacro:macro>
   <xacro:macro name="module_cage" params="prefix parent *origin">
 		<joint name="${prefix}module_cage_joint" type="fixed">

File: rb_theron_description/urdf/pole/mcq_pole.urdf.xacro (robot description, xacro)
@@ -2,9 +2,9 @@
 <robot name="simple_pole"
   xmlns:xacro="http://www.ros.org/wiki/xacro">
-	<macro name="box_inertia_robot" params="m x y z">
+	<xacro:macro name="box_inertia_robot" params="m x y z">
 	        <inertia  ixx="${m*(y*y+z*z)/12}" ixy = "0" ixz = "0"
 	                  iyy="${m*(x*x+z*z)/12}" iyz = "0"
 	                  izz="${m*(x*x+z*z)/12}" />
-	</macro>
+	</xacro:macro>
   <xacro:macro name="mcq_pole" params="prefix parent *origin">
 		<joint name="${prefix}pole_joint" type="fixed">

File: rb_theron_description/urdf/pole/simple_pole.urdf.xacro (robot description, xacro)
@@ -2,9 +2,9 @@
 <robot name="simple_pole"
   xmlns:xacro="http://www.ros.org/wiki/xacro">
-	<macro name="box_inertia_robot" params="m x y z">
+	<xacro:macro name="box_inertia_robot" params="m x y z">
 	        <inertia  ixx="${m*(y*y+z*z)/12}" ixy = "0" ixz = "0"
 	                  iyy="${m*(x*x+z*z)/12}" iyz = "0"
 	                  izz="${m*(x*x+z*z)/12}" />
-	</macro>
+	</xacro:macro>
   <xacro:macro name="simple_pole" params="prefix parent *origin">
 		<joint name="${prefix}pole_joint" type="fixed">

File: rb_theron_description/urdf/rocker/mcq_prototype_rocker.urdf.xacro (robot description, xacro)
@@ -18,5 +18,5 @@
       <parent link="${parent}"/>
       <child link="${prefix}support"/>
-      <insert_block name="origin" />
+      <xacro:insert_block name="origin" />
       <axis xyz="0 1 0" rpy="0 0 ${M_PI}" />
       <limit effort="100" velocity="100"/>
@@ -26,5 +26,5 @@
       <parent link="${parent}"/>
       <child link="${prefix}rsupport"/>
-      <insert_block name="origin" />
+      <xacro:insert_block name="origin" />
       <axis xyz="0 1 0" rpy="0 0 ${M_PI}" />
       <limit lower="-0.5" upper="0.5" effort="100" velocity="100"/>

File: rb_theron_description/urdf/wheels/castor.urdf.xacro (robot description, xacro)
@@ -3,9 +3,9 @@
   <xacro:property name="M_PI" value="3.1415926535897931" />
   <!-- Caster support parameters -->
-  <property name="caster_support_mass" value="1.5" /> <!-- in kg-->
+  <xacro:property name="caster_support_mass" value="1.5" /> <!-- in kg-->
   <!-- Caster wheel parameters -->
-  <property name="caster_radius" value="0.050" />
-  <property name="caster_height" value="0.025" />
-  <property name="caster_mass" value="0.25" /> <!-- in kg-->
+  <xacro:property name="caster_radius" value="0.050" />
+  <xacro:property name="caster_height" value="0.025" />
+  <xacro:property name="caster_mass" value="0.25" /> <!-- in kg-->
   <!-- Caster wheel offset-->
   <xacro:property name="caster_wheel_offset_x" value="-0.033" />
@@ -23,5 +23,5 @@
       <parent link="${parent}"/>
       <child link="${prefix}support"/>
-      <insert_block name="origin" />
+      <xacro:insert_block name="origin" />
       <axis xyz="0 0 1" rpy="0 ${M_PI} 0" />
       <limit effort="100" velocity="100"/>
@@ -58,5 +58,5 @@
        <parent link="${parent}"/>
        <child link="${prefix}wheel"/>
-       <insert_block name="origin" />
+       <xacro:insert_block name="origin" />
        <axis xyz="0 1 0" rpy="0 0 0" />
        <limit effort="100" velocity="100"/>

Commit message: rs_bpeal einbau

File: rb_theron_description/robots/rb_theron.urdf.xacro (robot description, xacro)
@@ -77,7 +77,10 @@
 		<origin xyz="0.250 0.0 0.1643" rpy="0 3.1416 3.1416"/>
 	</xacro:sensor_sick_nanoscan3>
-	<xacro:sensor_rs_lidar_16 prefix="$(arg prefix)top_laser" parent="$(arg prefix)base_link" prefix_topic="top_laser" min_angle="-3.1416" max_angle="3.1416">
+	<!--<xacro:sensor_rs_lidar_16 prefix="$(arg prefix)top_laser" parent="$(arg prefix)base_link" prefix_topic="top_laser" min_angle="-3.1416" max_angle="3.1416">
 		<origin xyz="0.214 0.0 0.275" rpy="-1.57079632679 0 -0.23"/>
-	</xacro:sensor_rs_lidar_16>
+	</xacro:sensor_rs_lidar_16>-->
+	<xacro:sensor_rs_bpearl prefix="$(arg prefix)top_laser"  parent="$(arg prefix)base_link" prefix_topic="top_laser" range_min="0.1" range_max="90" hfov="360" samples="1200" vfov="90.0" lasers="32" fps="15" gpu="false">
+            <origin xyz="0.414 0.0 0.275" rpy="0 0 0"/>
+        </xacro:sensor_rs_bpearl>
 	<!-- <xacro:sensor_sick_nanoscan3 prefix="$(arg prefix)back_laser" parent="$(arg prefix)base_link" prefix_topic="back_laser" min_angle="-1.8107619" max_angle="1.8107619">
 		<origin xyz="-0.250 0.0 0.1643" rpy="0 3.1416 0"/>

Commit message: rs_bpearl positioning

File: rb_theron_description/robots/rb_theron.urdf.xacro (robot description, xacro)
@@ -81,5 +81,5 @@
 	</xacro:sensor_rs_lidar_16>-->
 	<xacro:sensor_rs_bpearl prefix="$(arg prefix)top_laser"  parent="$(arg prefix)base_link" prefix_topic="top_laser" range_min="0.1" range_max="90" hfov="360" samples="1200" vfov="90.0" lasers="32" fps="15" gpu="false">
-            <origin xyz="0.414 0.0 0.275" rpy="0 0 0"/>
+            <origin xyz="0.26 0.151 1.3" rpy="-1.570796326795 0 -1.570796326795"/>
         </xacro:sensor_rs_bpearl>
 	<!-- <xacro:sensor_sick_nanoscan3 prefix="$(arg prefix)back_laser" parent="$(arg prefix)base_link" prefix_topic="back_laser" min_angle="-1.8107619" max_angle="1.8107619">

Commit message: Repositioning lidar and theron cage

File: rb_theron_description/robots/rb_theron.urdf.xacro (robot description, xacro)
@@ -81,5 +81,5 @@
 	</xacro:sensor_rs_lidar_16>-->
 	<xacro:sensor_rs_bpearl prefix="$(arg prefix)top_laser"  parent="$(arg prefix)base_link" prefix_topic="top_laser" range_min="0.1" range_max="90" hfov="360" samples="1200" vfov="90.0" lasers="32" fps="15" gpu="false">
-            <origin xyz="0.26 0.151 1.3" rpy="-1.570796326795 0 -1.570796326795"/>
+            <origin xyz="0.28 -0.159 1.22" rpy="-1.570796326795 0 -1.570796326795"/>
         </xacro:sensor_rs_bpearl>
 	<!-- <xacro:sensor_sick_nanoscan3 prefix="$(arg prefix)back_laser" parent="$(arg prefix)base_link" prefix_topic="back_laser" min_angle="-1.8107619" max_angle="1.8107619">
@@ -89,5 +89,5 @@
 	<xacro:include filename="$(find rb_theron_description)/urdf/module_cage/module_cage.urdf.xacro" />
 	<xacro:module_cage prefix="$(arg prefix)module_cage" parent="$(arg prefix)base_link">
-		<origin xyz="-0.18 -0.1997 0.2225" rpy="0 0 1.570796326794896619"/>
+		<origin xyz="0.35 -0.0 -0.075" rpy="0 0 1.570796326794896619"/>
 	</xacro:module_cage>
 </robot>
